File: PCB/quad_pcb/quad_pcb.kicad_sch (KiCad schematic)
At the start: 15 parts, among them J1 Screw_Terminal_01x02, U1 ESP32-S3-WROOM-1, U2 AP63203WU, U3 AMS1117-3.3

Commit message: PWM controllers added, connected to added drvs
Parts:
- added C10, C12, C14, C16, C17, C18, C22, C23, C24, C28, C29, C30: .1uF / 50V, symbol Device:C
- added C11, C13, C15, C19, C20, C21, C25, C26, C27, C31, C32, C33: 22uF / 63V, symbol Device:C_Polarized
- added C34, C35: 10uF, symbol Device:C
- added D1, D2, D3, D4, D5, D6, D7, D8: BLUE, symbol Device:LED
- added J10, J11, J12, J13, J2, J3, J4, J5, J6, J7, J8, J9: Screw_Terminal_01x02, symbol Connector:Screw_Terminal_01x02
- added J14, J15, J16, J17: Screw_Terminal_01x03, symbol Connector:Screw_Terminal_01x03
- added R10, R11, R12, R13, R2, R3, R4, R5, R6, R7, R8, R9: 15k, symbol Device:R
- added R14, R15, R16, R17, R18, R19, R20, R21, R22, R23, R24, R25, R26, R27: 10k, symbol Device:R
- added R28, R29, R30, R31, R32, R33, R34, R35: 10, symbol Device:R
- added U10, U11, U12, U13, U14, U15, U4, U5, U6, U7, U8, U9: DRV8871DDA, Package_SO:Texas_HTSOP-8-1EP_3.9x4.9mm_P1.27mm_EP2.95x4.9mm_Mask2.4x3.1mm_ThermalVias, symbol Driver_Motor:DRV8871DDA
- added U16, U17: PCA9685PW, Package_SO:TSSOP-28_4.4x9.7mm_P0.65mm, symbol Driver_LED:PCA9685PW
Connections:
- net 12V: now also C10.1, C11.1, C12.1, C13.1, C14.1, C15.1, C16.1, C17.1, C18.1, C19.1, C20.1, C21.1, C22.1, C23.1, C24.1, C25.1, C26.1, C27.1, C28.1, C29.1, C30.1, C31.1, C32.1, C33.1, U10.5 (VM), U11.5 (VM), U12.5 (VM), U13.5 (VM), U14.5 (VM), U15.5 (VM), U4.5 (VM), U5.5 (VM), U6.5 (VM), U7.5 (VM), U8.5 (VM), U9.5 (VM)
- net 3V3: now also C34.1, C35.1, J14.1 (Pin_1), J15.3 (Pin_3), J16.1 (Pin_1), J17.3 (Pin_3), R26.1, U16.28 (VDD), U17.1 (A0), U17.28 (VDD)
- net GND: now also C10.2, C11.2, C12.2, C13.2, C14.2, C15.2, C16.2, C17.2, C18.2, C19.2, C20.2, C21.2, C22.2, C23.2, C24.2, C25.2, C26.2, C27.2, C28.2, C29.2, C30.2, C31.2, C32.2, C33.2, C34.2, C35.2, D1.1 (K), D2.1 (K), D3.1 (K), D4.1 (K), D5.1 (K), D6.1 (K), D7.1 (K), D8.1 (K), R10.2, R11.2, R12.2, R13.2, R14.2, R15.2, R16.2, R17.2, R18.2, R19.2, R2.2, R20.2, R21.2, R22.2, R23.2, R24.2, R25.2, R26.2, R27.2, R3.2, R4.2, R5.2, R6.2, R7.2, R8.2, R9.2, U10.1 (GND), U10.7 (GND), U10.9 (GND), U11.1 (GND), U11.7 (GND), U11.9 (GND), U12.1 (GND), U12.7 (GND), U12.9 (GND), U13.1 (GND), U13.7 (GND), U13.9 (GND), U14.1 (GND), U14.7 (GND), U14.9 (GND), U15.1 (GND), U15.7 (GND), U15.9 (GND), U16.14 (VSS), U16.25 (EXTCLK), U17.14 (VSS), U17.25 (EXTCLK), U4.1 (GND), U4.7 (GND), U4.9 (GND), U5.1 (GND), U5.7 (GND), U5.9 (GND), U6.1 (GND), U6.7 (GND), U6.9 (GND), U7.1 (GND), U7.7 (GND), U7.9 (GND), U8.1 (GND), U8.7 (GND), U8.9 (GND), U9.1 (GND), U9.7 (GND), U9.9 (GND)
- new net: R19.1, U16.4 (A3)
- new net: R9.1, U11.4 (ILIM)
- new net: J9.1 (Pin_1), U11.6 (OUT1)
- new net: J9.2 (Pin_2), U11.8 (OUT2)
- new net: R24.1, U17.2 (A1)
- new net: D7.2 (A), R34.1
- new net: R34.2, U17.16 (LED9)
- new net: R13.1, U15.4 (ILIM)
- new net: D6.2 (A), R33.1
- new net: J5.1 (Pin_1), U7.6 (OUT1)
- new net: J5.2 (Pin_2), U7.8 (OUT2)
- new net: R25.1, U17.5 (A4)
- new net: R10.1, U12.4 (ILIM)
- new net: J10.1 (Pin_1), U12.6 (OUT1)
- new net: J10.2 (Pin_2), U12.8 (OUT2)
- new net: J6.1 (Pin_1), U8.6 (OUT1)
- new net: J6.2 (Pin_2), U8.8 (OUT2)
- new net: R11.1, U13.4 (ILIM)
- new net: J11.1 (Pin_1), U13.6 (OUT1)
- new net: J11.2 (Pin_2), U13.8 (OUT2)
- new net: J7.1 (Pin_1), U9.6 (OUT1)
- new net: J7.2 (Pin_2), U9.8 (OUT2)
- new net: R4.1, U6.4 (ILIM)
- new net: J4.1 (Pin_1), U6.6 (OUT1)
- new net: J4.2 (Pin_2), U6.8 (OUT2)
- new net: J12.1 (Pin_1), U14.6 (OUT1)
- new net: J12.2 (Pin_2), U14.8 (OUT2)
- new net: R3.1, U5.4 (ILIM)
- new net: J3.1 (Pin_1), U5.6 (OUT1)
- new net: J3.2 (Pin_2), U5.8 (OUT2)
- new net: R8.1, U10.4 (ILIM)
- new net: J8.1 (Pin_1), U10.6 (OUT1)
- new net: J8.2 (Pin_2), U10.8 (OUT2)
- new net: R16.1, U16.1 (A0)
- new net: J13.1 (Pin_1), U15.6 (OUT1)
- new net: J13.2 (Pin_2), U15.8 (OUT2)
- new net: D4.2 (A), R31.1
- new net: R31.2, U17.19 (LED12)
- new net: R6.1, U8.4 (ILIM)
- new net: D2.2 (A), R29.1
- new net: J2.1 (Pin_1), U4.6 (OUT1)
- new net: J2.2 (Pin_2), U4.8 (OUT2)
- new net: D8.2 (A), R35.1
- new net: R15.1, U17.23 (~{OE})
- new net: R5.1, U7.4 (ILIM)
- new net: D1.2 (A), R28.1
- new net: R28.2, U17.22 (LED15)
- new net: D3.2 (A), R30.1
- new net: R30.2, U17.20 (LED13)
- new net: R35.2, U17.15 (LED8)
- new net: R7.1, U9.4 (ILIM)
- new net: R12.1, U14.4 (ILIM)
- new net: R21.1, U16.24 (A5)
- new net: R22.1, U17.3 (A2)
- new net: D5.2 (A), R32.1
- new net: R32.2, U17.18 (LED11)
- new net: R23.1, U17.24 (A5)
- new net: R2.1, U4.4 (ILIM)
- new net: R20.1, U16.5 (A4)
- new net: R18.1, U16.3 (A2)
- new net: R29.2, U17.21 (LED14)
- new net: R33.2, U17.17 (LED10)
- new net: R27.1, U17.4 (A3)
- new net: R17.1, U16.2 (A1)
- new net: R14.1, U16.23 (~{OE})
- new net LEG_1_A1: U16.15 (LED8), U4.3 (IN1)
- new net LEG_1_A2: U16.16 (LED9), U4.2 (IN2)
- new net LEG_1_B1: U16.17 (LED10), U5.3 (IN1)
- new net LEG_1_B2: U16.18 (LED11), U5.2 (IN2)
- new net LEG_2_A1: U16.19 (LED12), U7.3 (IN1)
- new net LEG_2_A2: U16.20 (LED13), U7.2 (IN2)
- new net LEG_2_B1: U16.21 (LED14), U8.3 (IN1)
- new net LEG_2_B2: U16.22 (LED15), U8.2 (IN2)
- new net LEG_3_A1: U10.3 (IN1), U17.6 (LED0)
- new net LEG_3_A2: U10.2 (IN2), U17.7 (LED1)
- new net LEG_3_B1: U11.3 (IN1), U17.8 (LED2)
- new net LEG_3_B2: U11.2 (IN2), U17.9 (LED3)
- new net LEG_4_A1: U13.3 (IN1), U17.10 (LED4)
- new net LEG_4_A2: U13.2 (IN2), U17.11 (LED5)
- new net LEG_4_B1: U14.3 (IN1), U17.12 (LED6)
- new net LEG_4_B2: U14.2 (IN2), U17.13 (LED7)
- new net LEG_HIP_1_1: U16.6 (LED0), U6.3 (IN1)
- new net LEG_HIP_1_2: U16.7 (LED1), U6.2 (IN2)
- new net LEG_HIP_2_1: U16.8 (LED2), U9.3 (IN1)
- new net LEG_HIP_2_2: U16.9 (LED3), U9.2 (IN2)
- new net LEG_HIP_3_1: U12.3 (IN1), U16.10 (LED4)
- new net LEG_HIP_3_2: U12.2 (IN2), U16.11 (LED5)
- new net LEG_HIP_4_1: U15.3 (IN1), U16.12 (LED6)
- new net LEG_HIP_4_2: U15.2 (IN2), U16.13 (LED7)
- new net SCL: U16.26 (SCL), U17.26 (SCL)
- new net SDA: U16.27 (SDA), U17.27 (SDA)
Other:
- note added: "0x40"
- note added: "0x41"
- moved on the sheet: C1, C2, C3, C4, C5, C6, C7, C8, C9, FB1, J1, R1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

Commit message: small changes
Parts:
- added R36, R37: 4.7k, symbol Device:R
Connections:
- net 3V3: now also R36.2, R37.2
- net GND: now also U1.1 (GND), U1.40 (GND), U1.41 (GND)
- net SCL: now also U1.24 (GPIO47/SPICLK_P/SUBSPICLK_P_DIFF), R36.1
- net SDA: now also U1.25 (GPIO48/SPICLK_N/SUBSPICLK_N_DIFF), R37.1
Other:
- moved on the sheet: C1, C2, C3, R1, U1
